File: tamtam_board/tamtam_board.kicad_pcb (KiCad board)
At the start: 2 copper layers, 56 parts, among them J1 Conn_02x03_Odd_Even, J10 Conn_01x03, J11 Conn_01x03, J12 Conn_01x03, J13 Conn_01x03, J14 Conn_01x03, J15 Conn_01x03, J16 Conn_01x03, J17 Conn_01x03, J18 Conn_01x03, J19 Conn_01x04, J2 Conn_01x03, J20 Conn_02x01, J21 Conn_01x02, J22 Conn_01x03, J23 Conn_01x03, J24 Conn_01x03, J25 Conn_01x03, J26 Conn_01x03, J27 Conn_01x04, J28 Conn_01x03, J29 Conn_01x03, J3 Conn_01x03, J30 Conn_01x03, J31 Conn_01x03, J32 Conn_01x03, J33 Conn_01x04, J34 Conn_01x04, J35 Conn_01x04, J36 Conn_01x04, J4 Conn_01x03, J5 Conn_01x03, J6 Conn_01x03, J7 Conn_01x03, J8 Conn_01x03, J9 Conn_01x03, Q1 IRF3205, U1 ATmega328P-AU, U2 SD20, Y1 Resonator, Y2 Crystal

Commit message: board finished
Parts:
- removed BZ1: Buzzer, Buzzer_Beeper:Buzzer_12x9.5RM7.6
- removed D1: LED, LED_SMD:LED_0603_1608Metric_Pad1.05x0.95mm_HandSolder
- removed J20: Conn_02x01, Connector_Phoenix_MC_HighVoltage:PhoenixContact_MCV_1,5_2-G-5.08_1x02_P5.08mm_Vertical
- removed J21: Conn_01x02, Connector_Phoenix_MC_HighVoltage:PhoenixContact_MCV_1,5_2-G-5.08_1x02_P5.08mm_Vertical
- removed J36: Conn_01x04, Connector_PinHeader_2.54mm:PinHeader_1x04_P2.54mm_Vertical
- removed J4, J5: Conn_01x03, Connector_PinHeader_2.54mm:PinHeader_1x03_P2.54mm_Vertical
- removed R4: 220, Resistor_SMD:R_0603_1608Metric_Pad1.05x0.95mm_HandSolder
- C2, C3, C4, R1, R2, R3, R6, R7, U1: moved to B.Cu
- J3: value Conn_01x03 -> Conn_02x01; footprint Connector_PinHeader_2.54mm:PinHeader_1x03_P2.54mm_Vertical -> Connector_PinHeader_2.54mm:PinHeader_2x01_P2.54mm_Vertical
- moved J29 170.9 mm to (70.2, 63.2)
- moved J3 166.7 mm to (55.9, 40.3)
- moved J23 158.8 mm to (66.6, 63.2)
- moved J16 156.7 mm to (77.4, 63.1)
- moved Y1 156.4 mm to (78.6, 59.0)
- moved J11 154.4 mm to (59.1, 30.5)
- moved J12 153.8 mm to (64.0, 30.5)
- moved J8 153.1 mm to (73.8, 63.2)
- moved J13 148.4 mm to (68.8, 30.5)
- moved J2 146.8 mm to (53.0, 30.8)
- moved R9 145.4 mm to (56.2, 35.3), turned to 270 degrees
- moved J30 144.2 mm to (88.3, 63.1)
- moved R8 142.6 mm to (56.3, 31.5), turned to 90 degrees
- moved J32 138.0 mm to (103.9, 44.4), turned to 90 degrees
- moved C4 134.2 mm to (80.1, 42.3), turned to 90 degrees
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Connections:
- J2 pad 1: PD2 -> V_LIPO
- J3 pad 1: PD3 -> +6V
- U1 pad 1: PD3 -> Net-(U1-Pad1)
- U1 pad 11: PD7 -> Net-(U1-Pad11)
- U1 pad 14: BZR -> Net-(U1-Pad14)
- U1 pad 2: PD4 -> Net-(U1-Pad2)
- U1 pad 32: PD2 -> Net-(U1-Pad32)
Routing:
- net +5V: track 0.00 -> 162.7 mm, vias 0 -> 4
- net GND: track 0.00 -> 156.0 mm, vias 0 -> 2
- net servos_GND: track 0.00 -> 108.4 mm
- net +6V: track 0.00 -> 91.8 mm
- net LVL_LIPO: track 0.00 -> 66.2 mm, vias 0 -> 4
- net ADC1: track 0.00 -> 65.7 mm, vias 0 -> 2
- net ADC2: track 0.00 -> 58.3 mm, vias 0 -> 2
- net ADC3: track 0.00 -> 52.4 mm, vias 0 -> 2
- net SERVO19: track 0.00 -> 47.4 mm, vias 0 -> 2
- net SERVO18: track 0.00 -> 46.7 mm
- net SERVO15: track 0.00 -> 45.1 mm
- net SERVO16: track 0.00 -> 44.5 mm
- net SCL: track 0.00 -> 44.4 mm
- net SERVO14: track 0.00 -> 44.3 mm
- net RST: track 0.00 -> 43.9 mm
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Other:
- board outline added: 61.5 x 44 mm
- board text added: "+5V"
- board text added: "1"
- board text added: "2"
- board text added: "3"
- board text added: "A"
- board text added: "ADC"
- board text added: "BT"
- board text added: "EYES"
- board text added: "G"
- board text added: "I2C"
- board text added: "L"
- board text added: "S0"
- board text added: "S10"
- board text added: "S14"
- board text added: "S15"
- board text added: "S19"
- board text added: "S4"
- board text added: "S5"
- board text added: "S9"
- board text added: "TamTam v1.0"
- board text added: "V"
- board text added: "by FioPio"
