File: tamtam_board/tamtam_board.sch (KiCad schematic (older format))
At the start: 2 parts

Commit message: little more done
Parts:
- added J? (x20): Conn_01x03, symbol Connector_Generic:Conn_01x03
- added R? (x3): 4k7, symbol Device:R
Connections:
- net +5V: now also R?.1, R?.1, R?.1
- net servos_GND: now also J?.3 (Pin_3), J?.3 (Pin_3), J?.3 (Pin_3), J?.3 (Pin_3), J?.3 (Pin_3), J?.3 (Pin_3), J?.3 (Pin_3), J?.3 (Pin_3), J?.3 (Pin_3), J?.3 (Pin_3), J?.3 (Pin_3), J?.3 (Pin_3), J?.3 (Pin_3), J?.3 (Pin_3), J?.3 (Pin_3), J?.3 (Pin_3), J?.3 (Pin_3), J?.3 (Pin_3), J?.3 (Pin_3), J?.3 (Pin_3)
- new net +6V: J?.2 (Pin_2), J?.2 (Pin_2), J?.2 (Pin_2), J?.2 (Pin_2), J?.2 (Pin_2), J?.2 (Pin_2), J?.2 (Pin_2), J?.2 (Pin_2), J?.2 (Pin_2), J?.2 (Pin_2), J?.2 (Pin_2), J?.2 (Pin_2), J?.2 (Pin_2), J?.2 (Pin_2), J?.2 (Pin_2), J?.2 (Pin_2), J?.2 (Pin_2), J?.2 (Pin_2), J?.2 (Pin_2), J?.2 (Pin_2)
- new net SCL: R?.2
- new net SDA: R?.2
- new net SERVO0: J?.1 (Pin_1)
- new net SERVO1: J?.1 (Pin_1)
- new net SERVO10: J?.1 (Pin_1)
- new net SERVO11: J?.1 (Pin_1)
- new net SERVO12: J?.1 (Pin_1)
- new net SERVO13: J?.1 (Pin_1)
- new net SERVO14: J?.1 (Pin_1)
- new net SERVO15: J?.1 (Pin_1)
- new net SERVO16: J?.1 (Pin_1)
- new net SERVO17: J?.1 (Pin_1)
- new net SERVO18: J?.1 (Pin_1)
- new net SERVO19: J?.1 (Pin_1)
- new net SERVO2: J?.1 (Pin_1)
- new net SERVO3: J?.1 (Pin_1)
- new net SERVO4: J?.1 (Pin_1), R?.2
- new net SERVO5: J?.1 (Pin_1)
- new net SERVO6: J?.1 (Pin_1)
- new net SERVO7: J?.1 (Pin_1)
- new net SERVO8: J?.1 (Pin_1)
- new net SERVO9: J?.1 (Pin_1)
Other:
- moved on the sheet: Q?

Commit message: some more work done
Parts:
- added C?: 100n, symbol Device:C
- added C? (x2): 22p, symbol Device:C
- added C?: 47u, symbol Device:C
- added D?: LED, symbol Device:LED
- added J?: Conn_01x02, symbol Connector_Generic:Conn_01x02
- added J?: Conn_01x04, symbol Connector_Generic:Conn_01x04
- added J?: Conn_02x03_Odd_Even, symbol Connector_Generic:Conn_02x03_Odd_Even
- added R? (x2): 10k, symbol Device:R
- added R?: 220, symbol Device:R
- added U?: SD20, symbol missing_components:SD20
- added Y?: Resonator, symbol Device:Resonator
- added Y?: Crystal, symbol Device:Crystal
Connections:
- net +5V: now also C?.1, C?.2, D?.2 (A), J?.2 (Pin_2), U?.1 (+5V), U?.20 (+5V)
- net GND: now also C?.1, C?.1, C?.2, J?.2 (Pin_2), J?.4 (Pin_4), J?.6 (Pin_6), R?.1, R?.2, U?.19 (GND), U?.8 (GND), Y?.2
- net SCL: now also U?.28 (PC5), U?.14 (SCL)
- net SDA: now also U?.27 (PC4), U?.15 (SDA)
- net SERVO0: now also U?.2 (SERVO_1)
- net SERVO1: now also U?.3 (SERVO_2)
- net SERVO10: now also U?.17 (SERVO_11)
- net SERVO11: now also U?.18 (SERVO_12)
- net SERVO12: now also U?.21 (SERVO_13)
- net SERVO13: now also U?.22 (SERVO_14)
- net SERVO14: now also U?.23 (SERVO_15)
- net SERVO15: now also U?.24 (SERVO_16)
- net SERVO16: now also U?.25 (SERVO_17)
- net SERVO17: now also U?.26 (SERVO_18)
- net SERVO18: now also U?.27 (SERVO_19)
- net SERVO19: now also U?.28 (SERVO_20)
- net SERVO2: now also U?.4 (SERVO_3)
- net SERVO3: now also U?.5 (SERVO_4)
- net SERVO4: now also U?.6 (SERVO_5)
- net SERVO5: now also U?.7 (SERVO_6)
- net SERVO6: now also U?.11 (SERVO_7)
- net SERVO7: now also U?.12 (SERVO_8)
- net SERVO8: now also U?.13 (SERVO_9)
- net SERVO9: now also U?.16 (SERVO_10)
- net servos_ON: now also U?.12 (PB0)
- net eyes_GREEN: now reaches U?.10 (PD6)
- net eyes_GREEN: now also J?.2 (Pin_2)
- net eyes_BLUE: now reaches U?.13 (PB1)
- net eyes_BLUE: now also J?.1 (Pin_1)
- net MOSI: now reaches U?.15 (PB3)
- net MOSI: now also J?.4 (Pin_4)
- net MISO: now reaches U?.16 (PB4)
- net MISO: now also J?.1 (Pin_1)
- net SCK: now reaches U?.17 (PB5)
- net SCK: now also J?.3 (Pin_3)
- net at U?.20 (AREF): now also C?.1
- net LVL_LIPO: now reaches U?.23 (PC0)
- net LVL_LIPO: now also R?.1, R?.1
- net RST: now reaches U?.29 (~RESET~/PC6)
- net RST: now also J?.5 (Pin_5)
- net at U?.7 (XTAL1/PB6): now also C?.2, Y?.1
- net at U?.8 (XTAL2/PB7): now also C?.2, Y?.2
- net eyes_RED: now reaches U?.9 (PD5)
- net eyes_RED: now also J?.3 (Pin_3)
- new net: U?.10 (OSC2), Y?.3
- new net: U?.9 (OSC1), Y?.1
- new net: D?.1 (K), R?.2
- new net V_LIPO: J?.1 (Pin_1), R?.2

Commit message: schematic finished
Parts:
- added BZ1: Buzzer, symbol Device:Buzzer
- added J11, J12, J13, J2, J3, J4, J5: Conn_01x03, symbol Connector_Generic:Conn_01x03
- added J19, J33, J34, J35, J36: Conn_01x04, symbol Connector_Generic:Conn_01x04
- added J20: Conn_02x01, symbol Connector_Generic:Conn_02x01
- added R3: 10k, symbol Device:R
- added R6: 1k, symbol Device:R
- added R7: 2k, symbol Device:R
- gave numbers to parts that had none: 39
Connections:
- net +5V: now also J11.3 (Pin_3), J12.3 (Pin_3), J13.3 (Pin_3), J19.1 (Pin_1), J2.3 (Pin_3), J20.2 (Pin_2), J3.3 (Pin_3), J33.1 (Pin_1), J34.1 (Pin_1), J35.1 (Pin_1), J36.1 (Pin_1), J4.3 (Pin_3), J5.3 (Pin_3)
- net +6V: now also J20.1 (Pin_1)
- net GND: now also BZ1.2 (+), J11.2 (Pin_2), J12.2 (Pin_2), J13.2 (Pin_2), J19.2 (Pin_2), J2.2 (Pin_2), J3.2 (Pin_2), J33.4 (Pin_4), J34.4 (Pin_4), J35.4 (Pin_4), J36.4 (Pin_4), J4.2 (Pin_2), J5.2 (Pin_2), R3.2, R7.2
- net SCL: now also J33.3 (Pin_3), J34.3 (Pin_3), J35.3 (Pin_3), J36.3 (Pin_3)
- net SDA: now also J33.2 (Pin_2), J34.2 (Pin_2), J35.2 (Pin_2), J36.2 (Pin_2)
- net servos_ON: now also R3.1
- net PD3: now reaches U1.1 (PD3)
- net PD3: now also J3.1 (Pin_1)
- net PD7: now reaches U1.11 (PD7)
- net PD7: now also J5.1 (Pin_1)
- net BZR: now reaches U1.14 (PB2)
- net BZR: now also BZ1.1 (-)
- net PD4: now reaches U1.2 (PD4)
- net PD4: now also J4.1 (Pin_1)
- net ADC1: now reaches U1.24 (PC1)
- net ADC1: now also J11.1 (Pin_1)
- net ADC2: now reaches U1.25 (PC2)
- net ADC2: now also J12.1 (Pin_1)
- net ADC3: now reaches U1.26 (PC3)
- net ADC3: now also J13.1 (Pin_1)
- net RX: now reaches U1.30 (PD0)
- net RX: now also J19.3 (Pin_3)
- net TX: now reaches U1.31 (PD1)
- net TX: now also R6.2
- net PD2: now reaches U1.32 (PD2)
- net PD2: now also J2.1 (Pin_1)
- new net: J19.4 (Pin_4), R6.1, R7.1
- no-connect marks 0 -> 2
Other:
- moved on the sheet: D1, J1, J21, J27, Q1, R1, R2, R4, R5, R8, R9

Commit message: schematic finished
Parts:
- BZ1: footprint (none) -> Buzzer_Beeper:Buzzer_12x9.5RM7.6
- C1, C2, C3, C4: footprint (none) -> Capacitor_SMD:C_0603_1608Metric_Pad1.05x0.95mm_HandSolder
- D1: footprint (none) -> LED_SMD:LED_0603_1608Metric_Pad1.05x0.95mm_HandSolder
- J1: footprint (none) -> Connector_PinHeader_2.54mm:PinHeader_2x03_P2.54mm_Vertical
- J10, J11, J12, J13, J14, J15, J16, J17, J18, J2, J22, J23, J24, J25, J26, J28, J29, J3, J30, J31, J32, J4, J5, J6, J7, J8, J9: footprint (none) -> Connector_PinHeader_2.54mm:PinHeader_1x03_P2.54mm_Vertical
- J19, J27, J33, J34, J35, J36: footprint (none) -> Connector_PinHeader_2.54mm:PinHeader_1x04_P2.54mm_Vertical
- J20, J21: footprint (none) -> Connector_Phoenix_MC_HighVoltage:PhoenixContact_MCV_1,5_2-G-5.08_1x02_P5.08mm_Vertical
- R1, R2, R3, R4, R5, R6, R7, R8, R9: footprint (none) -> Resistor_SMD:R_0603_1608Metric_Pad1.05x0.95mm_HandSolder
- U2: footprint (none) -> Package_DIP:DIP-28_W7.62mm_Socket_LongPads
- Y1: footprint (none) -> Crystal:Resonator-3Pin_W7.0mm_H2.5mm
- Y2: footprint (none) -> Crystal:Crystal_HC49-4H_Vertical

Commit message: board finished
Parts:
- removed BZ1: Buzzer, Buzzer_Beeper:Buzzer_12x9.5RM7.6, symbol Device:Buzzer
- removed D1: LED, LED_SMD:LED_0603_1608Metric_Pad1.05x0.95mm_HandSolder, symbol Device:LED
- removed J20: Conn_02x01, Connector_Phoenix_MC_HighVoltage:PhoenixContact_MCV_1,5_2-G-5.08_1x02_P5.08mm_Vertical, symbol Connector_Generic:Conn_02x01
- removed J21: Conn_01x02, Connector_Phoenix_MC_HighVoltage:PhoenixContact_MCV_1,5_2-G-5.08_1x02_P5.08mm_Vertical, symbol Connector_Generic:Conn_01x02
- removed J3, J4, J5: Conn_01x03, Connector_PinHeader_2.54mm:PinHeader_1x03_P2.54mm_Vertical, symbol Connector_Generic:Conn_01x03
- removed J36: Conn_01x04, Connector_PinHeader_2.54mm:PinHeader_1x04_P2.54mm_Vertical, symbol Connector_Generic:Conn_01x04
- removed R4: 220, Resistor_SMD:R_0603_1608Metric_Pad1.05x0.95mm_HandSolder, symbol Device:R
- added J3: Conn_02x01, Connector_PinHeader_2.54mm:PinHeader_2x01_P2.54mm_Vertical, symbol Connector_Generic:Conn_02x01
Connections:
- net +6V: now also J3.1 (Pin_1)
- net GND: now also J3.2 (Pin_2)
- net V_LIPO: now also J2.1 (Pin_1)
- net BZR: no longer names the net of U1.14 (PB2)
- net PD2: no longer names the net of U1.32 (PD2)
- net PD2: no longer J2.1 (Pin_1)
- net PD3: no longer names the net of U1.1 (PD3)
- net PD4: no longer names the net of U1.2 (PD4)
- net PD7: no longer names the net of U1.11 (PD7)
- no-connect marks 2 -> 7
